File: RS485_LoadSwitch/Channel.kicad_sch (KiCad schematic)
At the start: 10 parts

Commit message: fix syntax
Changed lines of the file:
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@@
   (paper "A4")
   (title_block (title "Load Channel: IRLZ44N + Flyback + TVS + INA180"))
-  (global_label (at 30 30) (text "+12V_RAIL"))
-  (global_label (at 30 35) (text "GND"))
-  (global_label (at 30 40) (text "CTRL_5V"))
+  (global_label "+12V_RAIL" (at 30 30 0))
+  (global_label "GND"       (at 30 35 0))
+  (global_label "CTRL_5V"   (at 30 40 0))
   (symbol (lib_id "Device:Q_NMOS_GDS") (at 90 50)
     (property "Reference" "Qx")(property "Value" "IRLZ44N")
@@
   (symbol (lib_id "Device:LED") (at 125 35) (property "Reference" "LEDx")(property "Value" "GREEN"))
   (symbol (lib_id "Device:R") (at 120 35) (property "Reference" "R_LED")(property "Value" "2.2k"))
-  (global_label (at 150 50) (text "OUT#"))
-  (global_label (at 150 70) (text "ADC_SNS#"))
+  (global_label "OUT#"      (at 150 50 0))
+  (global_label "ADC_SNS#"  (at 150 70 0))
 )

Commit message: fix
Changed lines of the file:
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@@
   (paper "A4")
   (title_block (title "Load Channel: IRLZ44N + Flyback + TVS + INA180"))
-  (global_label "+12V_RAIL" (at 30 30 0))
-  (global_label "GND"       (at 30 35 0))
-  (global_label "CTRL_5V"   (at 30 40 0))
-  (symbol (lib_id "Device:Q_NMOS_GDS") (at 90 50)
+  (global_label "+12V_RAIL" (at 30 30 0) (shape input))
+  (global_label "GND"       (at 30 35 0) (shape input))
+  (global_label "CTRL_5V"   (at 30 40 0) (shape input))
+  (symbol (lib_id "Device:Q_NMOS_GDS") (at 90 50 0)
     (property "Reference" "Qx")(property "Value" "IRLZ44N")
   )
-  (symbol (lib_id "Device:R") (at 80 45) (property "Reference" "R_G")(property "Value" "22"))
-  (symbol (lib_id "Device:R") (at 80 55) (property "Reference" "R_PD")(property "Value" "100k"))
-  (symbol (lib_id "Diode:D_Schottky") (at 110 45)
+  (symbol (lib_id "Device:R") (at 80 45 0) (property "Reference" "R_G")(property "Value" "22"))
+  (symbol (lib_id "Device:R") (at 80 55 0) (property "Reference" "R_PD")(property "Value" "100k"))
+  (symbol (lib_id "Diode:D_Schottky") (at 110 45 0)
     (property "Reference" "D_FREE")(property "Value" "STPS3L60")
   )
-  (symbol (lib_id "Diode:TVS") (at 115 50)
+  (symbol (lib_id "Diode:TVS") (at 115 50 0)
     (property "Reference" "D_TVS")(property "Value" "SMBJ33A")
   )
-  (symbol (lib_id "Device:R") (at 90 65) (property "Reference" "R_SHUNT")(property "Value" "0.05R 1W"))
-  (symbol (lib_id "Device:U") (at 120 65) (property "Reference" "U_SNS")(property "Value" "INA180A1"))
-  (symbol (lib_id "Connector:Conn_01x02") (at 140 45)
+  (symbol (lib_id "Device:R") (at 90 65 0) (property "Reference" "R_SHUNT")(property "Value" "0.05R 1W"))
+  (symbol (lib_id "Device:U") (at 120 65 0) (property "Reference" "U_SNS")(property "Value" "INA180A1"))
+  (symbol (lib_id "Connector:Conn_01x02") (at 140 45 0)
     (property "Reference" "J_OUTx")(property "Value" "+12V / OUTx")
     (property "Footprint" "TerminalBlock_Phoenix:TerminalBlock_Phoenix_MSTBA_2_5.08mm")
   )
-  (symbol (lib_id "Device:LED") (at 125 35) (property "Reference" "LEDx")(property "Value" "GREEN"))
-  (symbol (lib_id "Device:R") (at 120 35) (property "Reference" "R_LED")(property "Value" "2.2k"))
-  (global_label "OUT#"      (at 150 50 0))
-  (global_label "ADC_SNS#"  (at 150 70 0))
+  (symbol (lib_id "Device:LED") (at 125 35 0) (property "Reference" "LEDx")(property "Value" "GREEN"))
+  (symbol (lib_id "Device:R") (at 120 35 0) (property "Reference" "R_LED")(property "Value" "2.2k"))
+  (global_label "OUT#"      (at 150 50 0) (shape output))
+  (global_label "ADC_SNS#"  (at 150 70 0) (shape output))
 )
