File: RS485_LoadSwitch/GateDriver.kicad_sch (KiCad schematic)
At the start: 1 part, among them U5 TC4468

Commit message: fix
Changed lines of the file:
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@@
   (paper "A4")
   (title_block (title "TC4468 Quad MOSFET Driver (5V)"))
-  (symbol (lib_id "Device:U") (at 80 60)
+  (symbol (lib_id "Device:U") (at 80 60 0)
     (property "Reference" "U5")(property "Value" "TC4468")
   )
-  (global_label (at 60 40) (text "+5V"))
-  (global_label (at 60 80) (text "GND"))
-  (global_label (at 110 45) (text "IN1"))
-  (global_label (at 110 50) (text "IN2"))
-  (global_label (at 110 55) (text "IN3"))
-  (global_label (at 110 60) (text "IN4"))
-  (global_label (at 130 45) (text "OUT1_5V"))
-  (global_label (at 130 50) (text "OUT2_5V"))
-  (global_label (at 130 55) (text "OUT3_5V"))
-  (global_label (at 130 60) (text "OUT4_5V"))
+  (global_label "+5V"      (at 60 40 0) (shape input))
+  (global_label "GND"      (at 60 80 0) (shape input))
+  (global_label "IN1"      (at 110 45 0) (shape input))
+  (global_label "IN2"      (at 110 50 0) (shape input))
+  (global_label "IN3"      (at 110 55 0) (shape input))
+  (global_label "IN4"      (at 110 60 0) (shape input))
+  (global_label "OUT1_5V"  (at 130 45 0) (shape output))
+  (global_label "OUT2_5V"  (at 130 50 0) (shape output))
+  (global_label "OUT3_5V"  (at 130 55 0) (shape output))
+  (global_label "OUT4_5V"  (at 130 60 0) (shape output))
 )
