File: RS485_LoadSwitch/MCU.kicad_sch (KiCad schematic)
At the start: 3 parts, among them U4 STM32F103C8T6

Commit message: fix syntax
Changed lines of the file:
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@@
     (property "Reference" "U4")(property "Value" "STM32F103C8T6")
   )
-  (global_label (at 80 40) (text "+3V3"))
-  (global_label (at 80 120) (text "GND"))
-  (global_label (at 140 50) (text "UART_TX"))
-  (global_label (at 140 55) (text "UART_RX"))
-  (global_label (at 140 60) (text "UART_DE"))
-  (global_label (at 140 65) (text "PWM1"))
-  (global_label (at 140 70) (text "PWM2"))
-  (global_label (at 140 75) (text "PWM3"))
-  (global_label (at 140 80) (text "PWM4"))
-  (global_label (at 140 85) (text "ADC_SNS1"))
-  (global_label (at 140 90) (text "ADC_SNS2"))
-  (global_label (at 140 95) (text "ADC_SNS3"))
-  (global_label (at 140 100) (text "ADC_SNS4"))
+  (global_label "+3V3"     (at 80 40 0))
+  (global_label "GND"      (at 80 120 0))
+  (global_label "UART_TX"  (at 140 50 0))
+  (global_label "UART_RX"  (at 140 55 0))
+  (global_label "UART_DE"  (at 140 60 0))
+  (global_label "PWM1"     (at 140 65 0))
+  (global_label "PWM2"     (at 140 70 0))
+  (global_label "PWM3"     (at 140 75 0))
+  (global_label "PWM4"     (at 140 80 0))
+  (global_label "ADC_SNS1" (at 140 85 0))
+  (global_label "ADC_SNS2" (at 140 90 0))
+  (global_label "ADC_SNS3" (at 140 95 0))
+  (global_label "ADC_SNS4" (at 140 100 0))
   (symbol (lib_id "Connector:Conn_01x05") (at 160 60)
     (property "Reference" "J_SWD")(property "Value" "SWD 1x5")

Commit message: fix
Changed lines of the file:
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@@
   (paper "A4")
   (title_block (title "MCU STM32F103C8T6 + SWD + DIP Addr"))
-  (symbol (lib_id "MCU_ST_STM32:STM32F103C8Tx") (at 100 80)
+  (symbol (lib_id "MCU_ST_STM32:STM32F103C8Tx") (at 100 80 0)
     (property "Reference" "U4")(property "Value" "STM32F103C8T6")
   )
-  (global_label "+3V3"     (at 80 40 0))
-  (global_label "GND"      (at 80 120 0))
-  (global_label "UART_TX"  (at 140 50 0))
-  (global_label "UART_RX"  (at 140 55 0))
-  (global_label "UART_DE"  (at 140 60 0))
-  (global_label "PWM1"     (at 140 65 0))
-  (global_label "PWM2"     (at 140 70 0))
-  (global_label "PWM3"     (at 140 75 0))
-  (global_label "PWM4"     (at 140 80 0))
-  (global_label "ADC_SNS1" (at 140 85 0))
-  (global_label "ADC_SNS2" (at 140 90 0))
-  (global_label "ADC_SNS3" (at 140 95 0))
-  (global_label "ADC_SNS4" (at 140 100 0))
-  (symbol (lib_id "Connector:Conn_01x05") (at 160 60)
+  (global_label "+3V3"     (at 80 40 0) (shape input))
+  (global_label "GND"      (at 80 120 0) (shape input))
+  (global_label "UART_TX"  (at 140 50 0) (shape output))
+  (global_label "UART_RX"  (at 140 55 0) (shape input))
+  (global_label "UART_DE"  (at 140 60 0) (shape output))
+  (global_label "PWM1"     (at 140 65 0) (shape output))
+  (global_label "PWM2"     (at 140 70 0) (shape output))
+  (global_label "PWM3"     (at 140 75 0) (shape output))
+  (global_label "PWM4"     (at 140 80 0) (shape output))
+  (global_label "ADC_SNS1" (at 140 85 0) (shape input))
+  (global_label "ADC_SNS2" (at 140 90 0) (shape input))
+  (global_label "ADC_SNS3" (at 140 95 0) (shape input))
+  (global_label "ADC_SNS4" (at 140 100 0) (shape input))
+  (symbol (lib_id "Connector:Conn_01x05") (at 160 60 0)
     (property "Reference" "J_SWD")(property "Value" "SWD 1x5")
   )
-  (symbol (lib_id "Connector_Generic:Conn_01x08") (at 160 90)
+  (symbol (lib_id "Connector_Generic:Conn_01x08") (at 160 90 0)
     (property "Reference" "SW_DIP")(property "Value" "DIP-8 Address")
   )
