File: RS485_LoadSwitch/Power.kicad_sch (KiCad schematic)
At the start: 12 parts, among them J1 PWR_IN (Vin+, GND, SHIELD), U1 LM2596S-5.0, U2 MCP1700-3302

Commit message: fix
Parts:
- D_BK: symbol Diode:D_Schottky -> Device:D_Schottky
Changed lines of the file:
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@@
   )
   (symbol (lib_id "Device:L") (at 160 50) (property "Reference" "L1")(property "Value" "33uH"))
-  (symbol (lib_id "Diode:D_Schottky") (at 160 60) (property "Reference" "D_BK")(property "Value" "MBR360"))
   (symbol (lib_id "Device:C") (at 120 70) (property "Reference" "CIN")(property "Value" "100uF/35V"))
+  (symbol (lib_id "Device:D_Schottky") (at 160 60) (property "Reference" "D_BK")(property "Value" "MBR360"))
   (symbol (lib_id "Device:C") (at 175 70) (property "Reference" "COUT1")(property "Value" "330uF/10V"))
   (symbol (lib_id "Device:C") (at 175 75) (property "Reference" "COUT2")(property "Value" "22uF"))

Commit message: update diode
Parts:
- D_BK: symbol Device:D_Schottky -> Diode:D_Schottky
Changed lines of the file:
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@@
   )
   (symbol (lib_id "Device:L") (at 160 50) (property "Reference" "L1")(property "Value" "33uH"))
+  (symbol (lib_id "Diode:D_Schottky") (at 160 60) (property "Reference" "D_BK")(property "Value" "MBR360"))
   (symbol (lib_id "Device:C") (at 120 70) (property "Reference" "CIN")(property "Value" "100uF/35V"))
-  (symbol (lib_id "Device:D_Schottky") (at 160 60) (property "Reference" "D_BK")(property "Value" "MBR360"))
   (symbol (lib_id "Device:C") (at 175 70) (property "Reference" "COUT1")(property "Value" "330uF/10V"))
   (symbol (lib_id "Device:C") (at 175 75) (property "Reference" "COUT2")(property "Value" "22uF"))

Commit message: fix syntax
Changed lines of the file:
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@@
     (property "Reference" "QRP")(property "Value" "IRF4905")
   )
-  (global_label (at 70 45) (text "+12V_IN"))
-  (global_label (at 90 45) (text "+12V_RAIL"))
-  (global_label (at 60 60) (text "GND"))
+  (global_label "+12V_IN"   (at 70 45 0))
+  (global_label "+12V_RAIL" (at 90 45 0))
+  (global_label "GND"       (at 60 60 0))
   (symbol (lib_id "Diode:TVS") (at 95 60)
     (property "Reference" "D_IN")(property "Value" "SMBJ24A")
@@
   (symbol (lib_id "Device:C") (at 175 70) (property "Reference" "COUT1")(property "Value" "330uF/10V"))
   (symbol (lib_id "Device:C") (at 175 75) (property "Reference" "COUT2")(property "Value" "22uF"))
-  (global_label (at 180 50) (text "+5V"))
-  (global_label (at 110 80) (text "GND"))
+  (global_label "+5V"  (at 180 50 0))
+  (global_label "GND"  (at 110 80 0))
   (symbol (lib_id "Regulator_Linear:MCP1700-3302") (at 200 50)
     (property "Reference" "U2")(property "Value" "MCP1700-3302")
@@
   (symbol (lib_id "Device:C") (at 195 70) (property "Reference" "C_LDO_IN")(property "Value" "1uF"))
   (symbol (lib_id "Device:C") (at 205 70) (property "Reference" "C_LDO_OUT")(property "Value" "1uF"))
-  (global_label (at 210 50) (text "+3V3"))
+  (global_label "+3V3" (at 210 50 0))
 )

Commit message: fix
Changed lines of the file:
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@@
   (paper "A4")
   (title_block (title "Power Block: Reverse Batt + Buck + LDO"))
-  (symbol (lib_id "Connector:Conn_01x03") (at 30 50)
+  (symbol (lib_id "Connector:Conn_01x03") (at 30 50 0)
     (property "Reference" "J1")(property "Value" "PWR_IN (Vin+, GND, SHIELD)")
     (property "Footprint" "TerminalBlock_Phoenix:TerminalBlock_Phoenix_MSTBA_3_5.08mm")
   )
-  (text "J1.1=+12V_IN  J1.2=GND  J1.3=SHIELD" (at 30 60))
-  (symbol (lib_id "Device:Q_PMOS_GDS") (at 80 50)
+  (text "J1.1=+12V_IN  J1.2=GND  J1.3=SHIELD" (at 30 60 0) (effects (font (size 1 1))))
+  (symbol (lib_id "Device:Q_PMOS_GDS") (at 80 50 0)
     (property "Reference" "QRP")(property "Value" "IRF4905")
   )
-  (global_label "+12V_IN"   (at 70 45 0))
-  (global_label "+12V_RAIL" (at 90 45 0))
-  (global_label "GND"       (at 60 60 0))
-  (symbol (lib_id "Diode:TVS") (at 95 60)
+  (global_label "+12V_IN"   (at 70 45 0) (shape input))
+  (global_label "+12V_RAIL" (at 90 45 0) (shape output))
+  (global_label "GND"       (at 60 60 0) (shape input))
+  (symbol (lib_id "Diode:TVS") (at 95 60 0)
     (property "Reference" "D_IN")(property "Value" "SMBJ24A")
   )
-  (symbol (lib_id "Regulator_Switching:LM2596S-5") (at 130 50)
+  (symbol (lib_id "Regulator_Switching:LM2596S-5") (at 130 50 0)
     (property "Reference" "U1")(property "Value" "LM2596S-5.0")
   )
-  (symbol (lib_id "Device:L") (at 160 50) (property "Reference" "L1")(property "Value" "33uH"))
-  (symbol (lib_id "Diode:D_Schottky") (at 160 60) (property "Reference" "D_BK")(property "Value" "MBR360"))
-  (symbol (lib_id "Device:C") (at 120 70) (property "Reference" "CIN")(property "Value" "100uF/35V"))
-  (symbol (lib_id "Device:C") (at 175 70) (property "Reference" "COUT1")(property "Value" "330uF/10V"))
-  (symbol (lib_id "Device:C") (at 175 75) (property "Reference" "COUT2")(property "Value" "22uF"))
-  (global_label "+5V"  (at 180 50 0))
-  (global_label "GND"  (at 110 80 0))
-  (symbol (lib_id "Regulator_Linear:MCP1700-3302") (at 200 50)
+  (symbol (lib_id "Device:L") (at 160 50 0) (property "Reference" "L1")(property "Value" "33uH"))
+  (symbol (lib_id "Diode:D_Schottky") (at 160 60 0) (property "Reference" "D_BK")(property "Value" "MBR360"))
+  (symbol (lib_id "Device:C") (at 120 70 0) (property "Reference" "CIN")(property "Value" "100uF/35V"))
+  (symbol (lib_id "Device:C") (at 175 70 0) (property "Reference" "COUT1")(property "Value" "330uF/10V"))
+  (symbol (lib_id "Device:C") (at 175 75 0) (property "Reference" "COUT2")(property "Value" "22uF"))
+  (global_label "+5V"  (at 180 50 0) (shape output))
+  (global_label "GND"  (at 110 80 0) (shape input))
+  (symbol (lib_id "Regulator_Linear:MCP1700-3302") (at 200 50 0)
     (property "Reference" "U2")(property "Value" "MCP1700-3302")
   )
-  (symbol (lib_id "Device:C") (at 195 70) (property "Reference" "C_LDO_IN")(property "Value" "1uF"))
-  (symbol (lib_id "Device:C") (at 205 70) (property "Reference" "C_LDO_OUT")(property "Value" "1uF"))
-  (global_label "+3V3" (at 210 50 0))
+  (symbol (lib_id "Device:C") (at 195 70 0) (property "Reference" "C_LDO_IN")(property "Value" "1uF"))
+  (symbol (lib_id "Device:C") (at 205 70 0) (property "Reference" "C_LDO_OUT")(property "Value" "1uF"))
+  (global_label "+3V3" (at 210 50 0) (shape output))
 )

Commit message: fix crash
Parts:
- D_BK: symbol Diode:D_Schottky -> Device:D_Schottky
Changed lines of the file:
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@@
   (paper "A4")
   (title_block (title "Power Block: Reverse Batt + Buck + LDO"))
-  (symbol (lib_id "Connector:Conn_01x03") (at 30 50 0)
-    (property "Reference" "J1")(property "Value" "PWR_IN (Vin+, GND, SHIELD)")
-    (property "Footprint" "TerminalBlock_Phoenix:TerminalBlock_Phoenix_MSTBA_3_5.08mm")
+  (symbol (lib_id "Connector:Conn_01x03") (at 30 50 0) (unit 1) (in_bom yes) (on_board yes)
+    (property "Reference" "J1" (at 30 48 0) (effects (font (size 1.27 1.27))))
+    (property "Value" "PWR_IN (Vin+, GND, SHIELD)" (at 30 52 0) (effects (font (size 1.27 1.27))))
+    (property "Footprint" "TerminalBlock_Phoenix:TerminalBlock_Phoenix_MSTBA_3_5.08mm" (at 30 54 0) (effects (font (size 1 1))))
   )
   (text "J1.1=+12V_IN  J1.2=GND  J1.3=SHIELD" (at 30 60 0) (effects (font (size 1 1))))
-  (symbol (lib_id "Device:Q_PMOS_GDS") (at 80 50 0)
-    (property "Reference" "QRP")(property "Value" "IRF4905")
+  (symbol (lib_id "Device:Q_PMOS_GDS") (at 80 50 0) (unit 1) (in_bom yes) (on_board yes)
+    (property "Reference" "QRP" (at 80 48 0) (effects (font (size 1.27 1.27))))
+    (property "Value" "IRF4905" (at 80 52 0) (effects (font (size 1.27 1.27))))
   )
-  (global_label "+12V_IN"   (at 70 45 0) (shape input))
-  (global_label "+12V_RAIL" (at 90 45 0) (shape output))
-  (global_label "GND"       (at 60 60 0) (shape input))
-  (symbol (lib_id "Diode:TVS") (at 95 60 0)
-    (property "Reference" "D_IN")(property "Value" "SMBJ24A")
+  (global_label "+12V_IN"   (at 70 45 0) (shape input)  (effects (font (size 1.27 1.27))) (uuid "pw000001-0000-4000-8000-000000000001"))
+  (global_label "+12V_RAIL" (at 90 45 0) (shape output) (effects (font (size 1.27 1.27))) (uuid "pw000001-0000-4000-8000-000000000002"))
+  (global_label "GND"       (at 60 60 0) (shape input)  (effects (font (size 1.27 1.27))) (uuid "pw000001-0000-4000-8000-000000000003"))
+  (symbol (lib_id "Diode:TVS") (at 95 60 0) (unit 1) (in_bom yes) (on_board yes)
+    (property "Reference" "D_IN" (at 95 58 0) (effects (font (size 1.27 1.27))))
+    (property "Value" "SMBJ24A" (at 95 62 0) (effects (font (size 1.27 1.27))))
   )
-  (symbol (lib_id "Regulator_Switching:LM2596S-5") (at 130 50 0)
-    (property "Reference" "U1")(property "Value" "LM2596S-5.0")
+  (symbol (lib_id "Regulator_Switching:LM2596S-5") (at 130 50 0) (unit 1) (in_bom yes) (on_board yes)
+    (property "Reference" "U1" (at 130 48 0) (effects (font (size 1.27 1.27))))
+    (property "Value" "LM2596S-5.0" (at 130 52 0) (effects (font (size 1.27 1.27))))
   )
-  (symbol (lib_id "Device:L") (at 160 50 0) (property "Reference" "L1")(property "Value" "33uH"))
-  (symbol (lib_id "Diode:D_Schottky") (at 160 60 0) (property "Reference" "D_BK")(property "Value" "MBR360"))
-  (symbol (lib_id "Device:C") (at 120 70 0) (property "Reference" "CIN")(property "Value" "100uF/35V"))
-  (symbol (lib_id "Device:C") (at 175 70 0) (property "Reference" "COUT1")(property "Value" "330uF/10V"))
-  (symbol (lib_id "Device:C") (at 175 75 0) (property "Reference" "COUT2")(property "Value" "22uF"))
-  (global_label "+5V"  (at 180 50 0) (shape output))
-  (global_label "GND"  (at 110 80 0) (shape input))
-  (symbol (lib_id "Regulator_Linear:MCP1700-3302") (at 200 50 0)
-    (property "Reference" "U2")(property "Value" "MCP1700-3302")
+  (symbol (lib_id "Device:L") (at 160 50 0) (unit 1) (in_bom yes) (on_board yes)
+    (property "Reference" "L1" (at 160 48 0) (effects (font (size 1.27 1.27))))
+    (property "Value" "33uH" (at 160 52 0) (effects (font (size 1.27 1.27))))
   )
-  (symbol (lib_id "Device:C") (at 195 70 0) (property "Reference" "C_LDO_IN")(property "Value" "1uF"))
-  (symbol (lib_id "Device:C") (at 205 70 0) (property "Reference" "C_LDO_OUT")(property "Value" "1uF"))
-  (global_label "+3V3" (at 210 50 0) (shape output))
+  (symbol (lib_id "Device:D_Schottky") (at 160 60 0) (unit 1) (in_bom yes) (on_board yes)
+    (property "Reference" "D_BK" (at 160 58 0) (effects (font (size 1.27 1.27))))
+    (property "Value" "MBR360" (at 160 62 0) (effects (font (size 1.27 1.27))))
+  )
+  (symbol (lib_id "Device:C") (at 120 70 0) (unit 1) (in_bom yes) (on_board yes)
+    (property "Reference" "CIN" (at 120 68 0) (effects (font (size 1.27 1.27))))
+    (property "Value" "100uF/35V" (at 120 72 0) (effects (font (size 1.27 1.27))))
+  )
+  (symbol (lib_id "Device:C") (at 175 70 0) (unit 1) (in_bom yes) (on_board yes)
+    (property "Reference" "COUT1" (at 175 68 0) (effects (font (size 1.27 1.27))))
+    (property "Value" "330uF/10V" (at 175 72 0) (effects (font (size 1.27 1.27))))
+  )
+  (symbol (lib_id "Device:C") (at 175 75 0) (unit 1) (in_bom yes) (on_board yes)
+    (property "Reference" "COUT2" (at 175 73 0) (effects (font (size 1.27 1.27))))
+    (property "Value" "22uF" (at 175 77 0) (effects (font (size 1.27 1.27))))
+  )
+  (global_label "+5V"  (at 180 50 0) (shape output) (effects (font (size 1.27 1.27))) (uuid "pw000001-0000-4000-8000-000000000004"))
+  (global_label "GND"  (at 110 80 0) (shape input)  (effects (font (size 1.27 1.27))) (uuid "pw000001-0000-4000-8000-000000000005"))
+  (symbol (lib_id "Regulator_Linear:MCP1700-3302") (at 200 50 0) (unit 1) (in_bom yes) (on_board yes)
+    (property "Reference" "U2" (at 200 48 0) (effects (font (size 1.27 1.27))))
+    (property "Value" "MCP1700-3302" (at 200 52 0) (effects (font (size 1.27 1.27))))
+  )
+  (symbol (lib_id "Device:C") (at 195 70 0) (unit 1) (in_bom yes) (on_board yes)
+    (property "Reference" "C_LDO_IN" (at 195 68 0) (effects (font (size 1.27 1.27))))
+    (property "Value" "1uF" (at 195 72 0) (effects (font (size 1.27 1.27))))
+  )
+  (symbol (lib_id "Device:C") (at 205 70 0) (unit 1) (in_bom yes) (on_board yes)
+    (property "Reference" "C_LDO_OUT" (at 205 68 0) (effects (font (size 1.27 1.27))))
+    (property "Value" "1uF" (at 205 72 0) (effects (font (size 1.27 1.27))))
+  )
+  (global_label "+3V3" (at 210 50 0) (shape output) (effects (font (size 1.27 1.27))) (uuid "pw000001-0000-4000-8000-000000000006"))
 )
