File: RS485_LoadSwitch/RS485.kicad_sch (KiCad schematic)
At the start: 6 parts, among them J2 RS485 (A,B,GND), U3 THVD1450

Commit message: fix syntax
Changed lines of the file:
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@@
     (property "Reference" "U3")(property "Value" "THVD1450")
   )
-  (global_label (at 45 40) (text "+5V"))
-  (global_label (at 45 60) (text "GND"))
-  (global_label (at 30 50) (text "UART_TX"))
-  (global_label (at 30 55) (text "UART_RX"))
-  (global_label (at 30 60) (text "UART_DE"))
-  (global_label (at 90 45) (text "RS485_A"))
-  (global_label (at 90 55) (text "RS485_B"))
+  (global_label "+5V"     (at 45 40 0))
+  (global_label "GND"     (at 45 60 0))
+  (global_label "UART_TX" (at 30 50 0))
+  (global_label "UART_RX" (at 30 55 0))
+  (global_label "UART_DE" (at 30 60 0))
+  (global_label "RS485_A" (at 90 45 0))
+  (global_label "RS485_B" (at 90 55 0))
   (symbol (lib_id "Device:R") (at 80 40) (property "Reference" "R_A_BIAS")(property "Value" "680"))
   (symbol (lib_id "Device:R") (at 80 60) (property "Reference" "R_B_BIAS")(property "Value" "680"))

Commit message: fix
Changed lines of the file:
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@@
   (paper "A4")
   (title_block (title "RS-485 Interface: THVD1450 + Protection"))
-  (symbol (lib_id "Interface_UART:MAX485") (at 60 50)
+  (symbol (lib_id "Interface_UART:MAX485") (at 60 50 0)
     (property "Reference" "U3")(property "Value" "THVD1450")
   )
-  (global_label "+5V"     (at 45 40 0))
-  (global_label "GND"     (at 45 60 0))
-  (global_label "UART_TX" (at 30 50 0))
-  (global_label "UART_RX" (at 30 55 0))
-  (global_label "UART_DE" (at 30 60 0))
-  (global_label "RS485_A" (at 90 45 0))
-  (global_label "RS485_B" (at 90 55 0))
-  (symbol (lib_id "Device:R") (at 80 40) (property "Reference" "R_A_BIAS")(property "Value" "680"))
-  (symbol (lib_id "Device:R") (at 80 60) (property "Reference" "R_B_BIAS")(property "Value" "680"))
-  (symbol (lib_id "Device:R") (at 90 50) (property "Reference" "R_TERM")(property "Value" "120"))
-  (symbol (lib_id "Diode:TVS") (at 110 50) (property "Reference" "D_RS485")(property "Value" "SM712"))
-  (symbol (lib_id "Connector:Conn_01x03") (at 140 50)
+  (global_label "+5V"     (at 45 40 0) (shape input))
+  (global_label "GND"     (at 45 60 0) (shape input))
+  (global_label "UART_TX" (at 30 50 0) (shape input))
+  (global_label "UART_RX" (at 30 55 0) (shape output))
+  (global_label "UART_DE" (at 30 60 0) (shape input))
+  (global_label "RS485_A" (at 90 45 0) (shape bidirectional))
+  (global_label "RS485_B" (at 90 55 0) (shape bidirectional))
+  (symbol (lib_id "Device:R") (at 80 40 0) (property "Reference" "R_A_BIAS")(property "Value" "680"))
+  (symbol (lib_id "Device:R") (at 80 60 0) (property "Reference" "R_B_BIAS")(property "Value" "680"))
+  (symbol (lib_id "Device:R") (at 90 50 0) (property "Reference" "R_TERM")(property "Value" "120"))
+  (symbol (lib_id "Diode:TVS") (at 110 50 0) (property "Reference" "D_RS485")(property "Value" "SM712"))
+  (symbol (lib_id "Connector:Conn_01x03") (at 140 50 0)
     (property "Reference" "J2")(property "Value" "RS485 (A,B,GND)")
     (property "Footprint" "TerminalBlock_Phoenix:TerminalBlock_Phoenix_MSTBA_3_5.08mm")
