File: RS485_LoadSwitch/RS485_LoadSwitch.kicad_sch (KiCad schematic)
At the start: 0 parts

Commit message: fix syntax
Other:
- note removed: "Tie nets via global labels. No explicit wires needed at top level."
Changed lines of the file:
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@@
     (comment 3 "TVS: SMBJ24A (input), SM712 (RS-485), SMBJ33A (outputs)")
   )
-  (global_label (shape input) (at 30 20) (text "+12V_IN"))
-  (global_label (shape input) (at 30 25) (text "+12V_RAIL"))
-  (global_label (shape input) (at 30 30) (text "+5V"))
-  (global_label (shape input) (at 30 35) (text "+3V3"))
-  (global_label (shape input) (at 30 40) (text "GND"))
+  (global_label "+12V_IN"   (at 30 20 0) (shape input))
+  (global_label "+12V_RAIL" (at 30 25 0) (shape input))
+  (global_label "+5V"       (at 30 30 0) (shape input))
+  (global_label "+3V3"      (at 30 35 0) (shape input))
+  (global_label "GND"       (at 30 40 0) (shape input))
   (sheet (at 30 60) (size 140 80)
     (property "Sheet name" "Power")
@@
     (pin (at 360 325) (name "ADC_SNS4") (shape output))
   )
-  (text "Tie nets via global labels. No explicit wires needed at top level.")
 )

Commit message: update sch
Other:
- sheet Channel1 ports: added ['uuid', '51111111-5555-5555-5555-000000000001'], ['uuid', '51111111-5555-5555-5555-000000000002'], ['uuid', '51111111-5555-5555-5555-000000000003'], ['uuid', '51111111-5555-5555-5555-000000000004'], ['uuid', '51111111-5555-5555-5555-000000000005']; removed ['uuid', '60'], ['uuid', '61'], ['uuid', '62'], ['uuid', '63'], ['uuid', '64']
- sheet Channel2 ports: added ['uuid', '52222222-5555-5555-5555-000000000001'], ['uuid', '52222222-5555-5555-5555-000000000002'], ['uuid', '52222222-5555-5555-5555-000000000003'], ['uuid', '52222222-5555-5555-5555-000000000004'], ['uuid', '52222222-5555-5555-5555-000000000005']; removed ['uuid', '70'], ['uuid', '71'], ['uuid', '72'], ['uuid', '73'], ['uuid', '74']
- sheet Channel3 ports: added ['uuid', '53333333-5555-5555-5555-000000000001'], ['uuid', '53333333-5555-5555-5555-000000000002'], ['uuid', '53333333-5555-5555-5555-000000000003'], ['uuid', '53333333-5555-5555-5555-000000000004'], ['uuid', '53333333-5555-5555-5555-000000000005']; removed ['uuid', '80'], ['uuid', '81'], ['uuid', '82'], ['uuid', '83'], ['uuid', '84']
- sheet Channel4 ports: added ['uuid', '54444444-5555-5555-5555-000000000001'], ['uuid', '54444444-5555-5555-5555-000000000002'], ['uuid', '54444444-5555-5555-5555-000000000003'], ['uuid', '54444444-5555-5555-5555-000000000004'], ['uuid', '54444444-5555-5555-5555-000000000005']; removed ['uuid', '90'], ['uuid', '91'], ['uuid', '92'], ['uuid', '93'], ['uuid', '94']
- sheet GateDriver ports: added ['uuid', '44444444-4444-4444-4444-000000000001'], ['uuid', '44444444-4444-4444-4444-000000000002'], ['uuid', '44444444-4444-4444-4444-000000000003'], ['uuid', '44444444-4444-4444-4444-000000000004'], ['uuid', '44444444-4444-4444-4444-000000000005'], ['uuid', '44444444-4444-4444-4444-000000000006'], ['uuid', '44444444-4444-4444-4444-000000000007'], ['uuid', '44444444-4444-4444-4444-000000000008'], ['uuid', '44444444-4444-4444-4444-000000000009'], ['uuid', '44444444-4444-4444-4444-00000000000a']; removed ['uuid', '40'], ['uuid', '41'], ['uuid', '42'], ['uuid', '43'], ['uuid', '44'], ['uuid', '45'], ['uuid', '46'], ['uuid', '47'], ['uuid', '48'], ['uuid', '49']
- sheet MCU ports: added ['uuid', '33333333-3333-3333-3333-000000000001'], ['uuid', '33333333-3333-3333-3333-000000000002'], ['uuid', '33333333-3333-3333-3333-000000000003'], ['uuid', '33333333-3333-3333-3333-000000000004'], ['uuid', '33333333-3333-3333-3333-000000000005'], ['uuid', '33333333-3333-3333-3333-000000000006'], ['uuid', '33333333-3333-3333-3333-000000000007'], ['uuid', '33333333-3333-3333-3333-000000000008'], ['uuid', '33333333-3333-3333-3333-000000000009'], ['uuid', '33333333-3333-3333-3333-00000000000a'], ['uuid', '33333333-3333-3333-3333-00000000000b'], ['uuid', '33333333-3333-3333-3333-00000000000c'], ['uuid', '33333333-3333-3333-3333-00000000000d']; removed ['uuid', '20'], ['uuid', '21'], ['uuid', '22'], ['uuid', '23'], ['uuid', '24'], ['uuid', '25'], ['uuid', '26'], ['uuid', '27'], ['uuid', '28'], ['uuid', '29'], ['uuid', '30'], ['uuid', '31'], ['uuid', '32']
- sheet Power ports: added ['uuid', '11111111-1111-1111-1111-000000000001'], ['uuid', '11111111-1111-1111-1111-000000000002'], ['uuid', '11111111-1111-1111-1111-000000000003'], ['uuid', '11111111-1111-1111-1111-000000000004'], ['uuid', '11111111-1111-1111-1111-000000000005']; removed ['uuid', '1'], ['uuid', '2'], ['uuid', '3'], ['uuid', '4'], ['uuid', '5']
- sheet RS485 ports: added ['uuid', '22222222-2222-2222-2222-000000000001'], ['uuid', '22222222-2222-2222-2222-000000000002'], ['uuid', '22222222-2222-2222-2222-000000000003'], ['uuid', '22222222-2222-2222-2222-000000000004'], ['uuid', '22222222-2222-2222-2222-000000000005'], ['uuid', '22222222-2222-2222-2222-000000000006'], ['uuid', '22222222-2222-2222-2222-000000000007']; removed ['uuid', '10'], ['uuid', '11'], ['uuid', '12'], ['uuid', '13'], ['uuid', '14'], ['uuid', '15'], ['uuid', '16']
Changed lines of the file:
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@@
     (property "Sheet name" "Power")
     (property "Sheet file" "Power.kicad_sch")
-    (pin (at 30 70) (name "+12V_IN") (shape input))
-    (pin (at 30 75) (name "GND") (shape input))
-    (pin (at 30 80) (name "+12V_RAIL") (shape output))
-    (pin (at 30 85) (name "+5V") (shape output))
-    (pin (at 30 90) (name "+3V3") (shape output))
+    (pin (at 30 70 0) (length 5.08) (name "+12V_IN")   (number "1") (shape input))
+    (pin (at 30 75 0) (length 5.08) (name "GND")        (number "2") (shape input))
+    (pin (at 30 80 0) (length 5.08) (name "+12V_RAIL")  (number "3") (shape output))
+    (pin (at 30 85 0) (length 5.08) (name "+5V")        (number "4") (shape output))
+    (pin (at 30 90 0) (length 5.08) (name "+3V3")       (number "5") (shape output))
   )
   (sheet (at 180 60) (size 140 60)
     (property "Sheet name" "RS485")
     (property "Sheet file" "RS485.kicad_sch")
-    (pin (at 180 70) (name "+5V") (shape input))
-    (pin (at 180 75) (name "GND") (shape input))
-    (pin (at 180 80) (name "UART_TX") (shape input))
-    (pin (at 180 85) (name "UART_RX") (shape output))
-    (pin (at 180 90) (name "UART_DE") (shape input))
-    (pin (at 180 95) (name "RS485_A") (shape bidirectional))
-    (pin (at 180 100) (name "RS485_B") (shape bidirectional))
+    (pin (at 180 70 0)  (length 5.08) (name "+5V")     (number "1") (shape input))
+    (pin (at 180 75 0)  (length 5.08) (name "GND")     (number "2") (shape input))
+    (pin (at 180 80 0)  (length 5.08) (name "UART_TX") (number "3") (shape input))
+    (pin (at 180 85 0)  (length 5.08) (name "UART_RX") (number "4") (shape output))
+    (pin (at 180 90 0)  (length 5.08) (name "UART_DE") (number "5") (shape input))
+    (pin (at 180 95 0)  (length 5.08) (name "RS485_A") (number "6") (shape bidirectional))
+    (pin (at 180 100 0) (length 5.08) (name "RS485_B") (number "7") (shape bidirectional))
   )
   (sheet (at 30 150) (size 150 90)
     (property "Sheet name" "MCU")
     (property "Sheet file" "MCU.kicad_sch")
-    (pin (at 30 160) (name "+3V3") (shape input))
-    (pin (at 30 165) (name "GND") (shape input))
-    (pin (at 30 170) (name "UART_TX") (shape output))
-    (pin (at 30 175) (name "UART_RX") (shape input))
-    (pin (at 30 180) (name "UART_DE") (shape output))
-    (pin (at 30 185) (name "PWM1") (shape output))
-    (pin (at 30 190) (name "PWM2") (shape output))
-    (pin (at 30 195) (name "PWM3") (shape output))
-    (pin (at 30 200) (name "PWM4") (shape output))
-    (pin (at 30 205) (name "ADC_SNS1") (shape input))
-    (pin (at 30 210) (name "ADC_SNS2") (shape input))
-    (pin (at 30 215) (name "ADC_SNS3") (shape input))
-    (pin (at 30 220) (name "ADC_SNS4") (shape input))
+    (pin (at 30 160 0) (length 5.08) (name "+3V3")     (number "1")  (shape input))
+    (pin (at 30 165 0) (length 5.08) (name "GND")      (number "2")  (shape input))
+    (pin (at 30 170 0) (length 5.08) (name "UART_TX")  (number "3")  (shape output))
+    (pin (at 30 175 0) (length 5.08) (name "UART_RX")  (number "4")  (shape input))
+    (pin (at 30 180 0) (length 5.08) (name "UART_DE")  (number "5")  (shape output))
+    (pin (at 30 185 0) (length 5.08) (name "PWM1")     (number "6")  (shape output))
+    (pin (at 30 190 0) (length 5.08) (name "PWM2")     (number "7")  (shape output))
+    (pin (at 30 195 0) (length 5.08) (name "PWM3")     (number "8")  (shape output))
+    (pin (at 30 200 0) (length 5.08) (name "PWM4")     (number "9")  (shape output))
+    (pin (at 30 205 0) (length 5.08) (name "ADC_SNS1") (number "10") (shape input))
+    (pin (at 30 210 0) (length 5.08) (name "ADC_SNS2") (number "11") (shape input))
+    (pin (at 30 215 0) (length 5.08) (name "ADC_SNS3") (number "12") (shape input))
+    (pin (at 30 220 0) (length 5.08) (name "ADC_SNS4") (number "13") (shape input))
   )
   (sheet (at 200 150) (size 120 70)
     (property "Sheet name" "GateDriver")
     (property "Sheet file" "GateDriver.kicad_sch")
-    (pin (at 200 160) (name "+5V") (shape input))
-    (pin (at 200 165) (name "GND") (shape input))
-    (pin (at 200 170) (name "IN1") (shape input))
-    (pin (at 200 175) (name "IN2") (shape input))
-    (pin (at 200 180) (name "IN3") (shape input))
-    (pin (at 200 185) (name "IN4") (shape input))
-    (pin (at 200 190) (name "OUT1_5V") (shape output))
-    (pin (at 200 195) (name "OUT2_5V") (shape output))
-    (pin (at 200 200) (name "OUT3_5V") (shape output))
-    (pin (at 200 205) (name "OUT4_5V") (shape output))
+    (pin (at 200 160 0) (length 5.08) (name "+5V")      (number "1") (shape input))
+    (pin (at 200 165 0) (length 5.08) (name "GND")      (number "2") (shape input))
+    (pin (at 200 170 0) (length 5.08) (name "IN1")      (number "3") (shape input))
+    (pin (at 200 175 0) (length 5.08) (name "IN2")      (number "4") (shape input))
+    (pin (at 200 180 0) (length 5.08) (name "IN3")      (number "5") (shape input))
+    (pin (at 200 185 0) (length 5.08) (name "IN4")      (number "6") (shape input))
+    (pin (at 200 190 0) (length 5.08) (name "OUT1_5V")  (number "7") (shape output))
+    (pin (at 200 195 0) (length 5.08) (name "OUT2_5V")  (number "8") (shape output))
+    (pin (at 200 200 0) (length 5.08) (name "OUT3_5V")  (number "9") (shape output))
+    (pin (at 200 205 0) (length 5.08) (name "OUT4_5V")  (number "10") (shape output))
   )
   (sheet (at 360 60) (size 120 70)
@@
     (property "Sheet file" "Channel.kicad_sch")
     (property "Channel" "1")
-    (pin (at 360 65) (name "+12V_RAIL") (shape input))
-    (pin (at 360 70) (name "GND") (shape input))
-    (pin (at 360 75) (name "CTRL_5V") (shape input))
-    (pin (at 360 80) (name "OUT1") (shape output))
-    (pin (at 360 85) (name "ADC_SNS1") (shape output))
+    (pin (at 360 65 0)  (length 5.08) (name "+12V_RAIL") (number "1") (shape input))
+    (pin (at 360 70 0)  (length 5.08) (name "GND")       (number "2") (shape input))
+    (pin (at 360 75 0)  (length 5.08) (name "CTRL_5V")   (number "3") (shape input))
+    (pin (at 360 80 0)  (length 5.08) (name "OUT1")      (number "4") (shape output))
+    (pin (at 360 85 0)  (length 5.08) (name "ADC_SNS1")  (number "5") (shape output))
   )
   (sheet (at 360 140) (size 120 70)
@@
     (property "Sheet file" "Channel.kicad_sch")
     (property "Channel" "2")
-    (pin (at 360 145) (name "+12V_RAIL") (shape input))
-    (pin (at 360 150) (name "GND") (shape input))
-    (pin (at 360 155) (name "CTRL_5V") (shape input))
-    (pin (at 360 160) (name "OUT2") (shape output))
-    (pin (at 360 165) (name "ADC_SNS2") (shape output))
+    (pin (at 360 145 0) (length 5.08) (name "+12V_RAIL") (number "1") (shape input))
+    (pin (at 360 150 0) (length 5.08) (name "GND")       (number "2") (shape input))
+    (pin (at 360 155 0) (length 5.08) (name "CTRL_5V")   (number "3") (shape input))
+    (pin (at 360 160 0) (length 5.08) (name "OUT2")      (number "4") (shape output))
+    (pin (at 360 165 0) (length 5.08) (name "ADC_SNS2")  (number "5") (shape output))
   )
   (sheet (at 360 220) (size 120 70)
@@
     (property "Sheet file" "Channel.kicad_sch")
     (property "Channel" "3")
-    (pin (at 360 225) (name "+12V_RAIL") (shape input))
-    (pin (at 360 230) (name "GND") (shape input))
-    (pin (at 360 235) (name "CTRL_5V") (shape input))
-    (pin (at 360 240) (name "OUT3") (shape output))
-    (pin (at 360 245) (name "ADC_SNS3") (shape output))
+    (pin (at 360 225 0) (length 5.08) (name "+12V_RAIL") (number "1") (shape input))
+    (pin (at 360 230 0) (length 5.08) (name "GND")       (number "2") (shape input))
+    (pin (at 360 235 0) (length 5.08) (name "CTRL_5V")   (number "3") (shape input))
+    (pin (at 360 240 0) (length 5.08) (name "OUT3")      (number "4") (shape output))
+    (pin (at 360 245 0) (length 5.08) (name "ADC_SNS3")  (number "5") (shape output))
   )
   (sheet (at 360 300) (size 120 70)
@@
     (property "Sheet file" "Channel.kicad_sch")
     (property "Channel" "4")
-    (pin (at 360 305) (name "+12V_RAIL") (shape input))
-    (pin (at 360 310) (name "GND") (shape input))
-    (pin (at 360 315) (name "CTRL_5V") (shape input))
-    (pin (at 360 320) (name "OUT4") (shape output))
-    (pin (at 360 325) (name "ADC_SNS4") (shape output))
+    (pin (at 360 305 0) (length 5.08) (name "+12V_RAIL") (number "1") (shape input))
+    (pin (at 360 310 0) (length 5.08) (name "GND")       (number "2") (shape input))
+    (pin (at 360 315 0) (length 5.08) (name "CTRL_5V")   (number "3") (shape input))
+    (pin (at 360 320 0) (length 5.08) (name "OUT4")      (number "4") (shape output))
+    (pin (at 360 325 0) (length 5.08) (name "ADC_SNS4")  (number "5") (shape output))
   )
 )

Commit message: fix
Other:
- sheet Channel1 ports: added none; removed ['uuid', '51111111-5555-5555-5555-000000000001'], ['uuid', '51111111-5555-5555-5555-000000000002'], ['uuid', '51111111-5555-5555-5555-000000000003'], ['uuid', '51111111-5555-5555-5555-000000000004'], ['uuid', '51111111-5555-5555-5555-000000000005']
- sheet Channel2 ports: added none; removed ['uuid', '52222222-5555-5555-5555-000000000001'], ['uuid', '52222222-5555-5555-5555-000000000002'], ['uuid', '52222222-5555-5555-5555-000000000003'], ['uuid', '52222222-5555-5555-5555-000000000004'], ['uuid', '52222222-5555-5555-5555-000000000005']
- sheet Channel3 ports: added none; removed ['uuid', '53333333-5555-5555-5555-000000000001'], ['uuid', '53333333-5555-5555-5555-000000000002'], ['uuid', '53333333-5555-5555-5555-000000000003'], ['uuid', '53333333-5555-5555-5555-000000000004'], ['uuid', '53333333-5555-5555-5555-000000000005']
- sheet Channel4 ports: added none; removed ['uuid', '54444444-5555-5555-5555-000000000001'], ['uuid', '54444444-5555-5555-5555-000000000002'], ['uuid', '54444444-5555-5555-5555-000000000003'], ['uuid', '54444444-5555-5555-5555-000000000004'], ['uuid', '54444444-5555-5555-5555-000000000005']
- sheet GateDriver ports: added none; removed ['uuid', '44444444-4444-4444-4444-000000000001'], ['uuid', '44444444-4444-4444-4444-000000000002'], ['uuid', '44444444-4444-4444-4444-000000000003'], ['uuid', '44444444-4444-4444-4444-000000000004'], ['uuid', '44444444-4444-4444-4444-000000000005'], ['uuid', '44444444-4444-4444-4444-000000000006'], ['uuid', '44444444-4444-4444-4444-000000000007'], ['uuid', '44444444-4444-4444-4444-000000000008'], ['uuid', '44444444-4444-4444-4444-000000000009'], ['uuid', '44444444-4444-4444-4444-00000000000a']
- sheet MCU ports: added none; removed ['uuid', '33333333-3333-3333-3333-000000000001'], ['uuid', '33333333-3333-3333-3333-000000000002'], ['uuid', '33333333-3333-3333-3333-000000000003'], ['uuid', '33333333-3333-3333-3333-000000000004'], ['uuid', '33333333-3333-3333-3333-000000000005'], ['uuid', '33333333-3333-3333-3333-000000000006'], ['uuid', '33333333-3333-3333-3333-000000000007'], ['uuid', '33333333-3333-3333-3333-000000000008'], ['uuid', '33333333-3333-3333-3333-000000000009'], ['uuid', '33333333-3333-3333-3333-00000000000a'], ['uuid', '33333333-3333-3333-3333-00000000000b'], ['uuid', '33333333-3333-3333-3333-00000000000c'], ['uuid', '33333333-3333-3333-3333-00000000000d']
- sheet Power ports: added none; removed ['uuid', '11111111-1111-1111-1111-000000000001'], ['uuid', '11111111-1111-1111-1111-000000000002'], ['uuid', '11111111-1111-1111-1111-000000000003'], ['uuid', '11111111-1111-1111-1111-000000000004'], ['uuid', '11111111-1111-1111-1111-000000000005']
- sheet RS485 ports: added none; removed ['uuid', '22222222-2222-2222-2222-000000000001'], ['uuid', '22222222-2222-2222-2222-000000000002'], ['uuid', '22222222-2222-2222-2222-000000000003'], ['uuid', '22222222-2222-2222-2222-000000000004'], ['uuid', '22222222-2222-2222-2222-000000000005'], ['uuid', '22222222-2222-2222-2222-000000000006'], ['uuid', '22222222-2222-2222-2222-000000000007']
Changed lines of the file:
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@@
     (property "Sheet name" "Power")
     (property "Sheet file" "Power.kicad_sch")
-    (pin (at 30 70 0) (length 5.08) (name "+12V_IN")   (number "1") (shape input))
-    (pin (at 30 75 0) (length 5.08) (name "GND")        (number "2") (shape input))
-    (pin (at 30 80 0) (length 5.08) (name "+12V_RAIL")  (number "3") (shape output))
-    (pin (at 30 85 0) (length 5.08) (name "+5V")        (number "4") (shape output))
-    (pin (at 30 90 0) (length 5.08) (name "+3V3")       (number "5") (shape output))
   )
   (sheet (at 180 60) (size 140 60)
     (property "Sheet name" "RS485")
     (property "Sheet file" "RS485.kicad_sch")
-    (pin (at 180 70 0)  (length 5.08) (name "+5V")     (number "1") (shape input))
-    (pin (at 180 75 0)  (length 5.08) (name "GND")     (number "2") (shape input))
-    (pin (at 180 80 0)  (length 5.08) (name "UART_TX") (number "3") (shape input))
-    (pin (at 180 85 0)  (length 5.08) (name "UART_RX") (number "4") (shape output))
-    (pin (at 180 90 0)  (length 5.08) (name "UART_DE") (number "5") (shape input))
-    (pin (at 180 95 0)  (length 5.08) (name "RS485_A") (number "6") (shape bidirectional))
-    (pin (at 180 100 0) (length 5.08) (name "RS485_B") (number "7") (shape bidirectional))
   )
   (sheet (at 30 150) (size 150 90)
     (property "Sheet name" "MCU")
     (property "Sheet file" "MCU.kicad_sch")
-    (pin (at 30 160 0) (length 5.08) (name "+3V3")     (number "1")  (shape input))
-    (pin (at 30 165 0) (length 5.08) (name "GND")      (number "2")  (shape input))
-    (pin (at 30 170 0) (length 5.08) (name "UART_TX")  (number "3")  (shape output))
-    (pin (at 30 175 0) (length 5.08) (name "UART_RX")  (number "4")  (shape input))
-    (pin (at 30 180 0) (length 5.08) (name "UART_DE")  (number "5")  (shape output))
-    (pin (at 30 185 0) (length 5.08) (name "PWM1")     (number "6")  (shape output))
-    (pin (at 30 190 0) (length 5.08) (name "PWM2")     (number "7")  (shape output))
-    (pin (at 30 195 0) (length 5.08) (name "PWM3")     (number "8")  (shape output))
-    (pin (at 30 200 0) (length 5.08) (name "PWM4")     (number "9")  (shape output))
-    (pin (at 30 205 0) (length 5.08) (name "ADC_SNS1") (number "10") (shape input))
-    (pin (at 30 210 0) (length 5.08) (name "ADC_SNS2") (number "11") (shape input))
-    (pin (at 30 215 0) (length 5.08) (name "ADC_SNS3") (number "12") (shape input))
-    (pin (at 30 220 0) (length 5.08) (name "ADC_SNS4") (number "13") (shape input))
   )
   (sheet (at 200 150) (size 120 70)
     (property "Sheet name" "GateDriver")
     (property "Sheet file" "GateDriver.kicad_sch")
-    (pin (at 200 160 0) (length 5.08) (name "+5V")      (number "1") (shape input))
-    (pin (at 200 165 0) (length 5.08) (name "GND")      (number "2") (shape input))
-    (pin (at 200 170 0) (length 5.08) (name "IN1")      (number "3") (shape input))
-    (pin (at 200 175 0) (length 5.08) (name "IN2")      (number "4") (shape input))
-    (pin (at 200 180 0) (length 5.08) (name "IN3")      (number "5") (shape input))
-    (pin (at 200 185 0) (length 5.08) (name "IN4")      (number "6") (shape input))
-    (pin (at 200 190 0) (length 5.08) (name "OUT1_5V")  (number "7") (shape output))
-    (pin (at 200 195 0) (length 5.08) (name "OUT2_5V")  (number "8") (shape output))
-    (pin (at 200 200 0) (length 5.08) (name "OUT3_5V")  (number "9") (shape output))
-    (pin (at 200 205 0) (length 5.08) (name "OUT4_5V")  (number "10") (shape output))
   )
   (sheet (at 360 60) (size 120 70)
@@
     (property "Sheet file" "Channel.kicad_sch")
     (property "Channel" "1")
-    (pin (at 360 65 0)  (length 5.08) (name "+12V_RAIL") (number "1") (shape input))
-    (pin (at 360 70 0)  (length 5.08) (name "GND")       (number "2") (shape input))
-    (pin (at 360 75 0)  (length 5.08) (name "CTRL_5V")   (number "3") (shape input))
-    (pin (at 360 80 0)  (length 5.08) (name "OUT1")      (number "4") (shape output))
-    (pin (at 360 85 0)  (length 5.08) (name "ADC_SNS1")  (number "5") (shape output))
   )
   (sheet (at 360 140) (size 120 70)
@@
     (property "Sheet file" "Channel.kicad_sch")
     (property "Channel" "2")
-    (pin (at 360 145 0) (length 5.08) (name "+12V_RAIL") (number "1") (shape input))
-    (pin (at 360 150 0) (length 5.08) (name "GND")       (number "2") (shape input))
-    (pin (at 360 155 0) (length 5.08) (name "CTRL_5V")   (number "3") (shape input))
-    (pin (at 360 160 0) (length 5.08) (name "OUT2")      (number "4") (shape output))
-    (pin (at 360 165 0) (length 5.08) (name "ADC_SNS2")  (number "5") (shape output))
   )
   (sheet (at 360 220) (size 120 70)
@@
     (property "Sheet file" "Channel.kicad_sch")
     (property "Channel" "3")
-    (pin (at 360 225 0) (length 5.08) (name "+12V_RAIL") (number "1") (shape input))
-    (pin (at 360 230 0) (length 5.08) (name "GND")       (number "2") (shape input))
-    (pin (at 360 235 0) (length 5.08) (name "CTRL_5V")   (number "3") (shape input))
-    (pin (at 360 240 0) (length 5.08) (name "OUT3")      (number "4") (shape output))
-    (pin (at 360 245 0) (length 5.08) (name "ADC_SNS3")  (number "5") (shape output))
   )
   (sheet (at 360 300) (size 120 70)
@@
     (property "Sheet file" "Channel.kicad_sch")
     (property "Channel" "4")
-    (pin (at 360 305 0) (length 5.08) (name "+12V_RAIL") (number "1") (shape input))
-    (pin (at 360 310 0) (length 5.08) (name "GND")       (number "2") (shape input))
-    (pin (at 360 315 0) (length 5.08) (name "CTRL_5V")   (number "3") (shape input))
-    (pin (at 360 320 0) (length 5.08) (name "OUT4")      (number "4") (shape output))
-    (pin (at 360 325 0) (length 5.08) (name "ADC_SNS4")  (number "5") (shape output))
   )
 )
