File: RS485_LoadSwitch/RS485_LoadSwitch.kicad_sch (KiCad schematic)
At the start: 0 parts

Commit message: fix crash
Changed lines of the file:
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@@
     (comment 3 "TVS: SMBJ24A (input), SM712 (RS-485), SMBJ33A (outputs)")
   )
-  (global_label "+12V_IN"   (at 30 20 0) (shape input))
-  (global_label "+12V_RAIL" (at 30 25 0) (shape input))
-  (global_label "+5V"       (at 30 30 0) (shape input))
-  (global_label "+3V3"      (at 30 35 0) (shape input))
-  (global_label "GND"       (at 30 40 0) (shape input))
+  (global_label "+12V_IN"   (at 30 20 0) (shape input) (effects (font (size 1.27 1.27))))
+  (global_label "+12V_RAIL" (at 30 25 0) (shape input) (effects (font (size 1.27 1.27))))
+  (global_label "+5V"       (at 30 30 0) (shape input) (effects (font (size 1.27 1.27))))
+  (global_label "+3V3"      (at 30 35 0) (shape input) (effects (font (size 1.27 1.27))))
+  (global_label "GND"       (at 30 40 0) (shape input) (effects (font (size 1.27 1.27))))
   (sheet (at 30 60) (size 140 80)
-    (property "Sheet name" "Power")
-    (property "Sheet file" "Power.kicad_sch")
+    (property "Sheet name" "Power" (at 32 58 0) (effects (font (size 1 1))))
+    (property "Sheet file" "Power.kicad_sch" (at 32 60 0) (effects (font (size 1 1))))
   )
   (sheet (at 180 60) (size 140 60)
-    (property "Sheet name" "RS485")
-    (property "Sheet file" "RS485.kicad_sch")
+    (property "Sheet name" "RS485" (at 182 58 0) (effects (font (size 1 1))))
+    (property "Sheet file" "RS485.kicad_sch" (at 182 60 0) (effects (font (size 1 1))))
   )
   (sheet (at 30 150) (size 150 90)
-    (property "Sheet name" "MCU")
-    (property "Sheet file" "MCU.kicad_sch")
+    (property "Sheet name" "MCU" (at 32 148 0) (effects (font (size 1 1))))
+    (property "Sheet file" "MCU.kicad_sch" (at 32 150 0) (effects (font (size 1 1))))
   )
   (sheet (at 200 150) (size 120 70)
-    (property "Sheet name" "GateDriver")
-    (property "Sheet file" "GateDriver.kicad_sch")
+    (property "Sheet name" "GateDriver" (at 202 148 0) (effects (font (size 1 1))))
+    (property "Sheet file" "GateDriver.kicad_sch" (at 202 150 0) (effects (font (size 1 1))))
   )
   (sheet (at 360 60) (size 120 70)
-    (property "Sheet name" "Channel1")
-    (property "Sheet file" "Channel.kicad_sch")
-    (property "Channel" "1")
+    (property "Sheet name" "Channel1" (at 362 58 0) (effects (font (size 1 1))))
+    (property "Sheet file" "Channel.kicad_sch" (at 362 60 0) (effects (font (size 1 1))))
+    (property "Channel" "1" (at 362 62 0) (effects (font (size 1 1))))
   )
   (sheet (at 360 140) (size 120 70)
-    (property "Sheet name" "Channel2")
-    (property "Sheet file" "Channel.kicad_sch")
-    (property "Channel" "2")
+    (property "Sheet name" "Channel2" (at 362 138 0) (effects (font (size 1 1))))
+    (property "Sheet file" "Channel.kicad_sch" (at 362 140 0) (effects (font (size 1 1))))
+    (property "Channel" "2" (at 362 142 0) (effects (font (size 1 1))))
   )
   (sheet (at 360 220) (size 120 70)
-    (property "Sheet name" "Channel3")
-    (property "Sheet file" "Channel.kicad_sch")
-    (property "Channel" "3")
+    (property "Sheet name" "Channel3" (at 362 218 0) (effects (font (size 1 1))))
+    (property "Sheet file" "Channel.kicad_sch" (at 362 220 0) (effects (font (size 1 1))))
+    (property "Channel" "3" (at 362 222 0) (effects (font (size 1 1))))
   )
   (sheet (at 360 300) (size 120 70)
-    (property "Sheet name" "Channel4")
-    (property "Sheet file" "Channel.kicad_sch")
-    (property "Channel" "4")
+    (property "Sheet name" "Channel4" (at 362 298 0) (effects (font (size 1 1))))
+    (property "Sheet file" "Channel.kicad_sch" (at 362 300 0) (effects (font (size 1 1))))
+    (property "Channel" "4" (at 362 302 0) (effects (font (size 1 1))))
   )
 )
