File: Opus-4.1/RS485_LoadSwitch.kicad_sch (KiCad schematic)
At the start: 81 parts, among them J1 PWR_IN, J2 RS485, J3 OUT1, J4 OUT2, J5 OUT3, J6 OUT4, J7 SWD, J8 SWD, U1 STM32F103C8T6, U5 INA181A1, U6 INA181A1, U7 INA181A1, U8 INA181A1, Y1 8MHz

Commit message: Add files via upload
Parts:
- added D18: CH2, LED_SMD:LED_0603_1608Metric, symbol Device:LED
- added D19: CH3, LED_SMD:LED_0603_1608Metric, symbol Device:LED
- added D20: CH4, LED_SMD:LED_0603_1608Metric, symbol Device:LED
- added R30, R31, R32: 1k, Resistor_SMD:R_0603_1608Metric, symbol Device:R
Connections:
- net +5V is gone; now on net +12V: J1.1 (Pin_1), J2.1 (Pin_1), J3.1 (Pin_1), J4.1 (Pin_1)
- net +12V: now also C20.1, C20.2, C21.1, C21.2, C22.1, C22.2, C23.1, C23.2, C24.1, C24.2, C25.1, C25.2, C26.1, C26.2, D17.1 (K), D17.2 (A), D6.2 (A2), D18.1 (K), D18.2 (A), D19.1 (K), D19.2 (A), D20.1 (K), D20.2 (A)
- net at J5.3 (GND): now also D14.2 (A)
- new net: D6.2 (A2), J4.2 (Pin_2)

Commit message: Add files via upload
Parts:
- added C27: 1uF/25V, Capacitor_SMD:C_0805_2012Metric, symbol Device:C
- added C28: 1nF, Capacitor_SMD:C_0603_1608Metric, symbol Device:C
- added F2, F3, F4, F5: 3.5A, Fuse:Fuse_1206_3216Metric, symbol Device:Fuse
- added L4: 100uH/15A, Inductor_THT:L_CommonMode_Toroid_Vertical_L21.0mm_W10.0mm_Px8.50mm_Py12.51mm_Wuerth_744823015, symbol Device:L_Coupled
- added R33: 3.0k, Resistor_SMD:R_0603_1608Metric, symbol Device:R
- added R34: 1.0k, Resistor_SMD:R_0603_1608Metric, symbol Device:R
- added R35: 10k, Resistor_SMD:R_0603_1608Metric, symbol Device:R
- added R36: 2.7k, Resistor_SMD:R_0603_1608Metric, symbol Device:R
- added R37: 2.2k, Resistor_SMD:R_0603_1608Metric, symbol Device:R
- added R38: 0.1R/5W, Resistor_THT:R_Axial_DIN0414_L11.9mm_D4.5mm_P15.24mm_Horizontal, symbol Device:R
- added RT1: 10k@25C, Resistor_SMD:R_0603_1608Metric, symbol Device:Thermistor_NTC
- added RV1: S14K20, Varistor:RV_Disc_D15.5mm_W4.2mm_P7.5mm, symbol Device:Varistor
- added TP5: IS1, TestPoint:TestPoint_Pad_D1.0mm, symbol Connector:TestPoint
- added TP6: G1, TestPoint:TestPoint_Pad_D1.0mm, symbol Connector:TestPoint
- added U10: LM393, Package_SO:SOIC-8_3.9x4.9mm_P1.27mm, symbol Comparator:LM393
- added U11: TL431, Package_TO_SOT_SMD:SOT-23, symbol Reference_Voltage:TL431LP
- added U9: TC4420CPA, Package_DIP:DIP-8_W7.62mm, symbol Driver_FET:TC4420
- C18: value 470uF/25V -> 470uF/35V; Ripple Current (none) -> 2A; Voltage (none) -> 35V
- F1: value 5A -> 15A; Manufacturer (none) -> Littelfuse; Part Number (none) -> 0154015.DR
- L2: value 33uH/5A -> 33uH/15A; Current Rating (none) -> 15A; DCR (none) -> 0.017Ω; Part Number (none) -> MSS1278-333MLD
Connections:
- net +12V: now also R9.2, R33.1, R35.2
- net at D13.2 (A): now also R38.2
- net at D13.1 (K), D14.1 (K), U1.18 (PB0)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: now also U1.37 (PA14), R35.1
- new net: D6.2 (A2), J4.2 (Pin_2)
- new net: R33.2, R34.1

Commit message: Add files via upload
Parts:
- added C29, C30, C31: 1uF/25V, Capacitor_SMD:C_0805_2012Metric, symbol Device:C
- added C32, C33, C34: 1nF, Capacitor_SMD:C_0603_1608Metric, symbol Device:C
- added C35: 100uF/25V, Capacitor_SMD:CP_Elec_6.3x5.4, symbol Device:CP
- added TP10: G2, TestPoint:TestPoint_Pad_D1.0mm, symbol Connector:TestPoint
- added TP11: G3, TestPoint:TestPoint_Pad_D1.0mm, symbol Connector:TestPoint
- added TP12: G4, TestPoint:TestPoint_Pad_D1.0mm, symbol Connector:TestPoint
- added TP13: OUT1, TestPoint:TestPoint_Pad_D1.5mm, symbol Connector:TestPoint
- added TP14: OUT2, TestPoint:TestPoint_Pad_D1.5mm, symbol Connector:TestPoint
- added TP15: OUT3, TestPoint:TestPoint_Pad_D1.5mm, symbol Connector:TestPoint
- added TP16: OUT4, TestPoint:TestPoint_Pad_D1.5mm, symbol Connector:TestPoint
- added TP7: IS2, TestPoint:TestPoint_Pad_D1.0mm, symbol Connector:TestPoint
- added TP8: IS3, TestPoint:TestPoint_Pad_D1.0mm, symbol Connector:TestPoint
- added TP9: IS4, TestPoint:TestPoint_Pad_D1.0mm, symbol Connector:TestPoint
- added U10, U11, U12: TC4420CPA, Package_DIP:DIP-8_W7.62mm, symbol Driver_FET:TC4420
- U10: symbol Comparator:LM393 -> Amplifier_Comparator:LM393
Connections:
- new net: D6.2 (A2), J4.2 (Pin_2)

Commit message: Add files via upload
Connections:
- new net: D6.2 (A2), J4.2 (Pin_2)
Other:
- note added: "- Under Q1-Q4 (MOSFETs)"
- note added: "- Under R5-R8 (sense resistors)"
- note added: "- Under U9-U12 (gate drivers)"
- note added: "CRITICAL: 3mm trace width for 3A paths"
- note added: "CRITICAL: Kelvin connections on R5-R8"
- note added: "CRITICAL: Star ground at C1"
- note added: "THERMAL VIAS REQUIRED:"
Changed lines of the file:
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@@
     (stroke (width 0) (type default))
     (uuid W_TVS_GND_CONNECT))
-  (wire (pts (xy 38.1 50.8) (xy 35.56 50.8))
-    (stroke (width 0) (type default))
-    (uuid W_J1_TO_MOV))
-  (wire (pts (xy 35.56 50.8) (xy 35.56 53.34))
-    (stroke (width 0) (type default))
-    (uuid W_MOV_TOP))
   (wire (pts (xy 35.56 60.96) (xy 35.56 71.12))
     (stroke (width 0) (type default))
@@
       (effects (font (size 1.27 1.27)) hide))
     (pin "1" (uuid TP6_GATE1-1)))
-  (wire (pts (xy 246.38 93.98) (xy 241.3 93.98))
-    (stroke (width 0) (type default))
-    (uuid W_PA0_TO_DRIVER1))
-  (wire (pts (xy 241.3 93.98) (xy 241.3 91.44))
-    (stroke (width 0) (type default))
-    (uuid W_DRIVER1_IN_ROUTE))
-  (wire (pts (xy 241.3 91.44) (xy 246.38 91.44))
-    (stroke (width 0) (type default))
-    (uuid W_TO_U9_IN))
   (wire (pts (xy 261.62 93.98) (xy 266.7 93.98))
     (stroke (width 0) (type default))
@@
     (stroke (width 0) (type default))
     (uuid W_C28_TO_SOURCE1))
+  (wire (pts (xy 38.1 50.8) (xy 35.56 45.72))
+    (stroke (width 0) (type default))
+    (uuid W_J1_POS_TO_CM_IN))
+  (wire (pts (xy 38.1 53.34) (xy 35.56 48.26))
+    (stroke (width 0) (type default))
+    (uuid W_J1_NEG_TO_CM_IN))
+  (wire (pts (xy 40.64 45.72) (xy 43.18 45.72))
+    (stroke (width 0) (type default))
+    (uuid W_CM_OUT_POS))
+  (wire (pts (xy 43.18 45.72) (xy 43.18 50.8))
+    (stroke (width 0) (type default))
+    (uuid W_CM_TO_MOV))
+  (wire (pts (xy 43.18 50.8) (xy 35.56 50.8))
+    (stroke (width 0) (type default))
+    (uuid W_TO_MOV_TOP))
+  (wire (pts (xy 35.56 50.8) (xy 35.56 53.34))
+    (stroke (width 0) (type default))
+    (uuid W_MOV_CONNECTION))
+  (wire (pts (xy 43.18 50.8) (xy 40.64 50.8))
+    (stroke (width 0) (type default))
+    (uuid W_MOV_TO_INRUSH))
+  (wire (pts (xy 40.64 48.26) (xy 43.18 48.26))
+    (stroke (width 0) (type default))
+    (uuid W_CM_OUT_NEG))
+  (wire (pts (xy 43.18 48.26) (xy 43.18 53.34))
+    (stroke (width 0) (type default))
+    (uuid W_CM_NEG_TO_GND))
+  (wire (pts (xy 43.18 53.34) (xy 50.8 53.34))
+    (stroke (width 0) (type default))
+    (uuid W_GND_PATH))
+  (wire (pts (xy 246.38 91.44) (xy 251.22 91.44))
+    (stroke (width 0) (type default))
+    (uuid W_TO_U9_PIN2))
+  (wire (pts (xy 251.22 91.44) (xy 251.22 93.98))
+    (stroke (width 0) (type default))
+    (uuid W_U9_PIN2_IN))
+  (wire (pts (xy 256.78 93.98) (xy 261.62 93.98))
+    (stroke (width 0) (type default))
+    (uuid W_U9_PIN6_OUT))
+  (wire (pts (xy 251.22 96.52) (xy 251.22 101.6))
+    (stroke (width 0) (type default))
+    (uuid W_U9_PIN3_GND))
+  (wire (pts (xy 251.22 101.6) (xy 254.0 101.6))
+    (stroke (width 0) (type default))
+    (uuid W_U9_GND_COMMON))
+  (wire (pts (xy 256.78 91.44) (xy 256.78 86.36))
+    (stroke (width 0) (type default))
+    (uuid W_U9_PIN7_VDD))
+  (wire (pts (xy 256.78 86.36) (xy 254.0 86.36))
+    (stroke (width 0) (type default))
+    (uuid W_U9_VDD_COMMON))
+  (wire (pts (xy 276.86 99.06) (xy 279.4 99.06))
+    (stroke (width 0) (type default))
+    (uuid W_C28_NEG))
+  (wire (pts (xy 279.4 99.06) (xy 279.4 101.6))
+    (stroke (width 0) (type default))
+    (uuid W_C28_TO_SOURCE))
+  (wire (pts (xy 279.4 99.06) (xy 279.4 96.52))
+    (stroke (width 0) (type default))
+    (uuid W_Q1_SOURCE))
+  (wire (pts (xy 279.4 96.52) (xy 264.16 96.52))
+    (stroke (width 0) (type default))
+    (uuid W_Q1_TO_SENSE))
+  (junction (at 312.42 81.28) (diameter 0) (color 0 0 0 0)
+    (uuid J_12V_MAIN))
+  (wire (pts (xy 312.42 81.28) (xy 254.0 81.28))
+    (stroke (width 0) (type default))
+    (uuid W_12V_TO_DRIVERS))
+  (wire (pts (xy 312.42 81.28) (xy 238.76 81.28))
+    (stroke (width 0) (type default))
+    (uuid W_12V_TO_BULK_CAP))
+  (wire (pts (xy 250.19 93.98) (xy 246.38 93.98))
+    (stroke (width 0) (type default))
+    (uuid W_R1_OUT))
+  (wire (pts (xy 246.38 93.98) (xy 241.3 93.98))
+    (stroke (width 0) (type default))
+    (uuid W_R1_TO_PA0))
+  (wire (pts (xy 241.3 93.98) (xy 220.98 93.98))
+    (stroke (width 0) (type default))
+    (uuid W_PA0_ROUTE))
+  (wire (pts (xy 220.98 93.98) (xy 220.98 58.42))
+    (stroke (width 0) (type default))
+    (uuid W_PA0_TO_MCU))
+  (wire (pts (xy 220.98 58.42) (xy 195.58 58.42))
+    (stroke (width 0) (type default))
+    (uuid W_PA0_CONNECT))
+  (text "THERMAL VIAS REQUIRED:" (at 250 160 0)
+    (effects (font (size 1.27 1.27)) (justify left)))
+  (text "- Under R5-R8 (sense resistors)" (at 250 162.5 0)
+    (effects (font (size 1.27 1.27)) (justify left)))
+  (text "- Under Q1-Q4 (MOSFETs)" (at 250 165 0)
+    (effects (font (size 1.27 1.27)) (justify left)))
+  (text "- Under U9-U12 (gate drivers)" (at 250 167.5 0)
+    (effects (font (size 1.27 1.27)) (justify left)))
+  (text "CRITICAL: 3mm trace width for 3A paths" (at 250 172.5 0)
+    (effects (font (size 1.27 1.27) bold) (justify left)))
+  (text "CRITICAL: Star ground at C1" (at 250 175 0)
+    (effects (font (size 1.27 1.27) bold) (justify left)))
+  (text "CRITICAL: Kelvin connections on R5-R8" (at 250 177.5 0)
+    (effects (font (size 1.27 1.27) bold) (justify left)))
   (symbol (lib_id "power:+12V") (at 307.34 86.36 0) (unit 1)
     (in_bom yes) (on_board yes) (dnp no)
